File: Electronics/EPS/eps.kicad_pcb (KiCad board)
At the start: 2 copper layers, 90 x 90 mm, 5 parts, among them J1 Conn_02x20_Odd_Even

Commit message: EPS Architecturing
Parts:
- H1, H2, H3, H4: value MountingHole_Pad -> M2.5
Connections:
- net /CAN2_N renamed /Connector/CAN2_N
- net /CAN2_P renamed /Connector/CAN2_P
- net /COMM_3V8 renamed /Connector/COM_3V8
- net /EPS_FALT renamed /Connector/COM_5V
- net /OBC_3V3_P renamed /Connector/OBC_3V3
- net /OBC_3V3_R renamed /Connector/OBC_5V
- net /PAYL_3V3 renamed /Connector/PAYL_3V3
- net /PAYL_5V renamed /Connector/PAYL_5V
- net /PAYL_CS renamed /Connector/PAYL_CS
- net /PAYL_FALT renamed /Connector/EPS_FALT
- net /PAYL_MISO renamed /Connector/PAYL_MISO
- net /PAYL_MOSI renamed /Connector/PAYL_MOSI
- net /PAYL_RQ renamed /Connector/PAYL_FALT
- net /PAYL_SCK renamed /Connector/PAYL_SCK
- net /PAYL_SCL renamed /Connector/PAYL_SCL
- net /PAYL_SDA renamed /Connector/PAYL_SDA
- net /RFU3 renamed /Connector/CAN1_P
- net /RFU6 renamed /Connector/CAN1_N
- J1 pad 10: /CAN1_N -> GND
- J1 pad 13: /RFU1 -> GND
- J1 pad 14: /RFU4 -> GND
- J1 pad 15: /RFU2 -> GND
- J1 pad 16: /RFU5 -> GND
- J1 pad 9: /CAN1_P -> GND
Routing:
- added copper zone on In2.Cu, net GND
Other:
- copper layers 2 -> 4
Changed lines of the file:
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@@
     (zones 0)
     (modules 5)
-    (nets 26)
+    (nets 20)
   )
   (page A4)
   (layers
     (0 F.Cu signal)
+    (1 In1.Cu mixed)
+    (2 In2.Cu power)
     (31 B.Cu signal)
     (32 B.Adhes user)
@@
     (solder_mask_min_width 0.25)
     (aux_axis_origin 0 0)
-    (visible_elements 7FFFFFFF)
+    (grid_origin 50 50)
+    (visible_elements 7FFFBFFF)
     (pcbplotparams
       (layerselection 0x010fc_ffffffff)
@@
   (net 0 "")
   (net 1 GND)
-  (net 2 /PAYL_5V)
-  (net 3 /PAYL_3V3)
-  (net 4 /PAYL_SCL)
-  (net 5 /PAYL_SDA)
-  (net 6 /PAYL_MISO)
-  (net 7 /PAYL_MOSI)
-  (net 8 /PAYL_CS)
-  (net 9 /PAYL_SCK)
-  (net 10 /PAYL_RQ)
-  (net 11 /PAYL_FALT)
-  (net 12 /CAN2_N)
-  (net 13 /CAN2_P)
-  (net 14 /RFU6)
-  (net 15 /RFU3)
-  (net 16 /RFU5)
-  (net 17 /RFU2)
-  (net 18 /RFU4)
-  (net 19 /RFU1)
-  (net 20 /CAN1_N)
-  (net 21 /CAN1_P)
-  (net 22 /EPS_FALT)
-  (net 23 /COMM_3V8)
-  (net 24 /OBC_3V3_R)
-  (net 25 /OBC_3V3_P)
+  (net 2 /Connector/PAYL_5V)
+  (net 3 /Connector/PAYL_3V3)
+  (net 4 /Connector/PAYL_SCL)
+  (net 5 /Connector/PAYL_SDA)
+  (net 6 /Connector/PAYL_MISO)
+  (net 7 /Connector/PAYL_MOSI)
+  (net 8 /Connector/PAYL_CS)
+  (net 9 /Connector/PAYL_SCK)
+  (net 10 /Connector/PAYL_FALT)
+  (net 11 /Connector/EPS_FALT)
+  (net 12 /Connector/CAN2_N)
+  (net 13 /Connector/CAN2_P)
+  (net 14 /Connector/CAN1_N)
+  (net 15 /Connector/CAN1_P)
+  (net 16 /Connector/COM_5V)
+  (net 17 /Connector/COM_3V8)
+  (net 18 /Connector/OBC_5V)
+  (net 19 /Connector/OBC_3V3)
   (net_class Default "This is the default net class."
     (clearance 0.2)
@@
     (uvia_dia 0.3)
     (uvia_drill 0.1)
-    (add_net /CAN1_N)
-    (add_net /CAN1_P)
-    (add_net /CAN2_N)
-    (add_net /CAN2_P)
-    (add_net /COMM_3V8)
-    (add_net /EPS_FALT)
-    (add_net /OBC_3V3_P)
-    (add_net /OBC_3V3_R)
-    (add_net /PAYL_3V3)
-    (add_net /PAYL_5V)
-    (add_net /PAYL_CS)
-    (add_net /PAYL_FALT)
-    (add_net /PAYL_MISO)
-    (add_net /PAYL_MOSI)
-    (add_net /PAYL_RQ)
-    (add_net /PAYL_SCK)
-    (add_net /PAYL_SCL)
-    (add_net /PAYL_SDA)
-    (add_net /RFU1)
-    (add_net /RFU2)
-    (add_net /RFU3)
-    (add_net /RFU4)
-    (add_net /RFU5)
-    (add_net /RFU6)
+    (add_net /Connector/CAN1_N)
+    (add_net /Connector/CAN1_P)
+    (add_net /Connector/CAN2_N)
+    (add_net /Connector/CAN2_P)
+    (add_net /Connector/COM_3V8)
+    (add_net /Connector/COM_5V)
+    (add_net /Connector/EPS_FALT)
+    (add_net /Connector/OBC_3V3)
+    (add_net /Connector/OBC_5V)
+    (add_net /Connector/PAYL_3V3)
+    (add_net /Connector/PAYL_5V)
+    (add_net /Connector/PAYL_CS)
+    (add_net /Connector/PAYL_FALT)
+    (add_net /Connector/PAYL_MISO)
+    (add_net /Connector/PAYL_MOSI)
+    (add_net /Connector/PAYL_SCK)
+    (add_net /Connector/PAYL_SCL)
+    (add_net /Connector/PAYL_SDA)
     (add_net GND)
   )
@@
     (fp_line (start -3.81 -1.27) (end 0.27 -1.27) (layer F.Fab) (width 0.1))
     (pad 40 thru_hole oval (at -2.54 48.26 90) (size 1.7 1.7) (drill 1) (layers *.Cu *.Mask)
-      (net 2 /PAYL_5V))
+      (net 2 /Connector/PAYL_5V))
     (pad 39 thru_hole oval (at 0 48.26 90) (size 1.7 1.7) (drill 1) (layers *.Cu *.Mask)
-      (net 3 /PAYL_3V3))
+      (net 3 /Connector/PAYL_3V3))
     (pad 38 thru_hole oval (at -2.54 45.72 90) (size 1.7 1.7) (drill 1) (layers *.Cu *.Mask)
       (net 1 GND))
@@
       (net 1 GND))
     (pad 36 thru_hole oval (at -2.54 43.18 90) (size 1.7 1.7) (drill 1) (layers *.Cu *.Mask)
-      (net 4 /PAYL_SCL))
+      (net 4 /Connector/PAYL_SCL))
     (pad 35 thru_hole oval (at 0 43.18 90) (size 1.7 1.7) (drill 1) (layers *.Cu *.Mask)
-      (net 5 /PAYL_SDA))
+      (net 5 /Connector/PAYL_SDA))
     (pad 34 thru_hole oval (at -2.54 40.64 90) (size 1.7 1.7) (drill 1) (layers *.Cu *.Mask)
       (net 1 GND))
@@
       (net 1 GND))
     (pad 32 thru_hole oval (at -2.54 38.1 90) (size 1.7 1.7) (drill 1) (layers *.Cu *.Mask)
-      (net 6 /PAYL_MISO))
+      (net 6 /Connector/PAYL_MISO))
     (pad 31 thru_hole oval (at 0 38.1 90) (size 1.7 1.7) (drill 1) (layers *.Cu *.Mask)
-      (net 7 /PAYL_MOSI))
+      (net 7 /Connector/PAYL_MOSI))
     (pad 30 thru_hole oval (at -2.54 35.56 90) (size 1.7 1.7) (drill 1) (layers *.Cu *.Mask)
-      (net 8 /PAYL_CS))
+      (net 8 /Connector/PAYL_CS))
     (pad 29 thru_hole oval (at 0 35.56 90) (size 1.7 1.7) (drill 1) (layers *.Cu *.Mask)
-      (net 9 /PAYL_SCK))
+      (net 9 /Connector/PAYL_SCK))
     (pad 28 thru_hole oval (at -2.54 33.02 90) (size 1.7 1.7) (drill 1) (layers *.Cu *.Mask)
       (net 1 GND))
@@
       (net 1 GND))
     (pad 26 thru_hole oval (at -2.54 30.48 90) (size 1.7 1.7) (drill 1) (layers *.Cu *.Mask)
-      (net 10 /PAYL_RQ))
+      (net 10 /Connector/PAYL_FALT))
     (pad 25 thru_hole oval (at 0 30.48 90) (size 1.7 1.7) (drill 1) (layers *.Cu *.Mask)
-      (net 11 /PAYL_FALT))
+      (net 11 /Connector/EPS_FALT))
     (pad 24 thru_hole oval (at -2.54 27.94 90) (size 1.7 1.7) (drill 1) (layers *.Cu *.Mask)
       (net 1 GND))
@@
       (net 1 GND))
     (pad 22 thru_hole oval (at -2.54 25.4 90) (size 1.7 1.7) (drill 1) (layers *.Cu *.Mask)
-      (net 12 /CAN2_N))
+      (net 12 /Connector/CAN2_N))
     (pad 21 thru_hole oval (at 0 25.4 90) (size 1.7 1.7) (drill 1) (layers *.Cu *.Mask)
-      (net 13 /CAN2_P))
+      (net 13 /Connector/CAN2_P))
     (pad 20 thru_hole oval (at -2.54 22.86 90) (size 1.7 1.7) (drill 1) (layers *.Cu *.Mask)
       (net 1 GND))
@@
       (net 1 GND))
     (pad 18 thru_hole oval (at -2.54 20.32 90) (size 1.7 1.7) (drill 1) (layers *.Cu *.Mask)
-      (net 14 /RFU6))
+      (net 14 /Connector/CAN1_N))
     (pad 17 thru_hole oval (at 0 20.32 90) (size 1.7 1.7) (drill 1) (layers *.Cu *.Mask)
-      (net 15 /RFU3))
+      (net 15 /Connector/CAN1_P))
     (pad 16 thru_hole oval (at -2.54 17.78 90) (size 1.7 1.7) (drill 1) (layers *.Cu *.Mask)
-      (net 16 /RFU5))
+      (net 1 GND))
     (pad 15 thru_hole oval (at 0 17.78 90) (size 1.7 1.7) (drill 1) (layers *.Cu *.Mask)
-      (net 17 /RFU2))
+      (net 1 GND))
     (pad 14 thru_hole oval (at -2.54 15.24 90) (size 1.7 1.7) (drill 1) (layers *.Cu *.Mask)
-      (net 18 /RFU4))
+      (net 1 GND))
     (pad 13 thru_hole oval (at 0 15.24 90) (size 1.7 1.7) (drill 1) (layers *.Cu *.Mask)
-      (net 19 /RFU1))
+      (net 1 GND))
     (pad 12 thru_hole oval (at -2.54 12.7 90) (size 1.7 1.7) (drill 1) (layers *.Cu *.Mask)
       (net 1 GND))
@@
       (net 1 GND))
     (pad 10 thru_hole oval (at -2.54 10.16 90) (size 1.7 1.7) (drill 1) (layers *.Cu *.Mask)
-      (net 20 /CAN1_N))
+      (net 1 GND))
     (pad 9 thru_hole oval (at 0 10.16 90) (size 1.7 1.7) (drill 1) (layers *.Cu *.Mask)
-      (net 21 /CAN1_P))
+      (net 1 GND))
     (pad 8 thru_hole oval (at -2.54 7.62 90) (size 1.7 1.7) (drill 1) (layers *.Cu *.Mask)
       (net 1 GND))
@@
       (net 1 GND))
     (pad 6 thru_hole oval (at -2.54 5.08 90) (size 1.7 1.7) (drill 1) (layers *.Cu *.Mask)
-      (net 22 /EPS_FALT))
+      (net 16 /Connector/COM_5V))
     (pad 5 thru_hole oval (at 0 5.08 90) (size 1.7 1.7) (drill 1) (layers *.Cu *.Mask)
-      (net 23 /COMM_3V8))
+      (net 17 /Connector/COM_3V8))
     (pad 4 thru_hole oval (at -2.54 2.54 90) (size 1.7 1.7) (drill 1) (layers *.Cu *.Mask)
       (net 1 GND))
@@
       (net 1 GND))
     (pad 2 thru_hole oval (at -2.54 0 90) (size 1.7 1.7) (drill 1) (layers *.Cu *.Mask)
-      (net 24 /OBC_3V3_R))
+      (net 18 /Connector/OBC_5V))
     (pad 1 thru_hole rect (at 0 0 90) (size 1.7 1.7) (drill 1) (layers *.Cu *.Mask)
-      (net 25 /OBC_3V3_P))
+      (net 19 /Connector/OBC_3V3))
     (model ${KISYS3DMOD}/Connector_PinSocket_2.54mm.3dshapes/PinSocket_2x20_P2.54mm_Vertical.wrl
       (at (xyz 0 0 0))
@@
       (effects (font (size 1 1) (thickness 0.15)))
     )
-    (fp_text value MountingHole_Pad (at 0 3.7) (layer F.Fab)
+    (fp_text value M2.5 (at 0 3.7) (layer F.Fab)
       (effects (font (size 1 1) (thickness 0.15)))
     )
@@
       (effects (font (size 1 1) (thickness 0.15)))
     )
-    (fp_text value MountingHole_Pad (at 0 3.7) (layer F.Fab)
+    (fp_text value M2.5 (at 0 3.7) (layer F.Fab)
       (effects (font (size 1 1) (thickness 0.15)))
     )
@@
       (effects (font (size 1 1) (thickness 0.15)))
     )
-    (fp_text value MountingHole_Pad (at 0 3.7) (layer F.Fab)
+    (fp_text value M2.5 (at 0 3.7) (layer F.Fab)
       (effects (font (size 1 1) (thickness 0.15)))
     )
@@
       (effects (font (size 1 1) (thickness 0.15)))
     )
-    (fp_text value MountingHole_Pad (at 0 3.7) (layer F.Fab)
+    (fp_text value M2.5 (at 0 3.7) (layer F.Fab)
       (effects (font (size 1 1) (thickness 0.15)))
     )
@@
   (gr_line (start 140 55) (end 140 135) (layer Edge.Cuts) (width 0.05))
   (gr_line (start 55 50) (end 135 50) (layer Edge.Cuts) (width 0.05))
+  (zone (net 1) (net_name GND) (layer In2.Cu) (hatch edge 0.508)
+    (connect_pads (clearance 0.508))
+    (min_thickness 0.254)
+    (fill yes (arc_segments 32) (thermal_gap 0.508) (thermal_bridge_width 1.016))
+    (polygon
+      (pts
+        (xy 140 140) (xy 50 140) (xy 50 50) (xy 140 50)
+      )
+    )
+  )
 )
