File: Electronics/Slice/slice.sch (KiCad schematic (older format))
At the start: 5 parts, among them J1 Conn_02x20_Odd_Even

Commit message: EPS Architecturing
Parts:
- removed H1, H2, H3, H4: MountingHole_Pad, MountingHole:MountingHole_2.7mm_M2.5_Pad, symbol Mechanical:MountingHole_Pad
- removed J1: Conn_02x20_Odd_Even, Connector_PinSocket_2.54mm:PinSocket_2x20_P2.54mm_Vertical, symbol Connector_Generic:Conn_02x20_Odd_Even
